Commit message: addeed camera

File: movit_config/config/ur.urdf (robot description, URDF)
Before this commit: robot ur, 24 links, 23 joints
Links:
- added link camera_head_color_frame
- added link camera_head_color_optical_frame
- added link camera_head_depth_frame
- added link camera_head_depth_optical_frame
- added link camera_head_infra1_frame
- added link camera_head_infra1_optical_frame
- added link camera_head_infra2_frame
- added link camera_head_infra2_optical_frame
- added link camera_head_link, mass 0.072; collision box size=0.02505 0.09 0.025; visual mesh filename=file:///home/darsh/ros2_ws/src/UR3_ROS2_PICK_AND_PLACE/inst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
- added link torso_link, mass 2.5; collision box size=0.15 0.10 0.06; collision cylinder length=0.6 radius=0.005
- link base_link_inertia: mass 4.0 -> 2.0; geometry collision mesh filename=package://ur_description/meshes/ur3/collision/base.stl; visual mesh filename=package://ur_description/meshes/ur3/visual/base.dae
- link forearm_link: mass 2.33 -> 1.26; geometry collision mesh filename=package://ur_description/meshes/ur3/collision/forearm.stl; visual mesh filename=package://ur_description/meshes/ur3/visual/forearm.dae
- link shoulder_link: mass 3.7 -> 2.0; geometry collision mesh filename=package://ur_description/meshes/ur3/collision/shoulder.stl; visual mesh filename=package://ur_description/meshes/ur3/visual/shoulder.dae
- link upper_arm_link: mass 8.393 -> 3.42; geometry collision mesh filename=package://ur_description/meshes/ur3/collision/upperarm.stl; visual mesh filename=package://ur_description/meshes/ur3/visual/upperarm.dae
- link wrist_1_link: mass 1.219 -> 0.8; geometry collision mesh filename=package://ur_description/meshes/ur3/collision/wrist1.stl; visual mesh filename=package://ur_description/meshes/ur3/visual/wrist1.dae
- link wrist_2_link: mass 1.219 -> 0.8; geometry collision mesh filename=package://ur_description/meshes/ur3/collision/wrist2.stl; visual mesh filename=package://ur_description/meshes/ur3/visual/wrist2.dae
- link wrist_3_link: mass 0.1879 -> 0.35; geometry collision mesh filename=package://ur_description/meshes/ur3/collision/wrist3.stl; visual mesh filename=package://ur_description/meshes/ur3/visual/wrist3.dae
Joints:
- added joint base_link_to_torso_link: type fixed, parent base_link, child torso_link, origin xyz=0.22 -0.30 0 rpy=0 0 0
- added joint camera_head_color_joint: type fixed, parent camera_head_link, child camera_head_color_frame, origin xyz=0 0.015 0 rpy=0 0 0
- added joint camera_head_color_optical_joint: type fixed, parent camera_head_color_frame, child camera_head_color_optical_frame, origin xyz=0 0 0 rpy=-1.5707963267948966 0 -1.5707963267948966
- added joint camera_head_depth_joint: type fixed, parent camera_head_link, child camera_head_depth_frame, origin xyz=0 0 0 rpy=0 0 0
- added joint camera_head_depth_optical_joint: type fixed, parent camera_head_depth_frame, child camera_head_depth_optical_frame, origin xyz=0 0 0 rpy=-1.5707963267948966 0 -1.5707963267948966
- added joint camera_head_infra1_joint: type fixed, parent camera_head_link, child camera_head_infra1_frame, origin xyz=0 0.0 0 rpy=0 0 0
- added joint camera_head_infra1_optical_joint: type fixed, parent camera_head_infra1_frame, child camera_head_infra1_optical_frame, origin xyz=0 0 0 rpy=-1.5707963267948966 0 -1.5707963267948966
- added joint camera_head_infra2_joint: type fixed, parent camera_head_link, child camera_head_infra2_frame, origin xyz=0 -0.05 0 rpy=0 0 0
- added joint camera_head_infra2_optical_joint: type fixed, parent camera_head_infra2_frame, child camera_head_infra2_optical_frame, origin xyz=0 0 0 rpy=-1.5707963267948966 0 -1.5707963267948966
- added joint camera_head_joint: type fixed, parent torso_link, child camera_head_link, origin xyz=0 0.01 0.50 rpy=0.0 0.4363323129985824 1.5707963267948966
- joint elbow_joint: limit lower=-3.141592653589793 upper=3.141592653589793 effort=150.0 velocity=3.141592653589793 -> lower=-3.141592653589793 upper=3.141592653589793 effort=28.0 velocity=3.141592653589793; origin xyz=-0.425 0 0 rpy=0 0 0 -> xyz=-0.24365 0 0 rpy=0 0 0
- joint shoulder_lift_joint: limit lower=-6.283185307179586 upper=6.283185307179586 effort=150.0 velocity=3.141592653589793 -> lower=-6.283185307179586 upper=6.283185307179586 effort=56.0 velocity=3.141592653589793
- joint shoulder_pan_joint: limit lower=-6.283185307179586 upper=6.283185307179586 effort=150.0 velocity=3.141592653589793 -> lower=-6.283185307179586 upper=6.283185307179586 effort=56.0 velocity=3.141592653589793; origin xyz=0 0 0.089159 rpy=0 0 0 -> xyz=0 0 0.1519 rpy=0 0 0
- joint wrist_1_joint: limit lower=-6.283185307179586 upper=6.283185307179586 effort=28.0 velocity=3.141592653589793 -> lower=-6.283185307179586 upper=6.283185307179586 effort=12.0 velocity=6.283185307179586; origin xyz=-0.39225 0 0.10915 rpy=0 0 0 -> xyz=-0.21325 0 0.11235 rpy=0 0 0
- joint wrist_2_joint: limit lower=-6.283185307179586 upper=6.283185307179586 effort=28.0 velocity=3.141592653589793 -> lower=-6.283185307179586 upper=6.283185307179586 effort=12.0 velocity=6.283185307179586; origin xyz=0 -0.09465 -1.941303950897609e-11 rpy=1.570796327 0 0 -> xyz=0 -0.08535 -1.750557762378351e-11 rpy=1.570796327 0 0
- joint wrist_3_joint: limit lower=-6.283185307179586 upper=6.283185307179586 effort=28.0 velocity=3.141592653589793 -> effort=12.0 velocity=6.283185307179586; origin xyz=0 0.0823 -1.688001216681175e-11 rpy=1.570796326589793 3.141592653589793 3.141592653589793 -> xyz=0 0.0819 -1.679797079540562e-11 rpy=1.570796326589793 3.141592653589793 3.141592653589793; type revolute -> continuous

File: ur_description/urdf/ur.urdf (robot description, URDF)
Before this commit: robot ur, 24 links, 23 joints
Links:
- added link camera_head_color_frame
- added link camera_head_color_optical_frame
- added link camera_head_depth_frame
- added link camera_head_depth_optical_frame
- added link camera_head_infra1_frame
- added link camera_head_infra1_optical_frame
- added link camera_head_infra2_frame
- added link camera_head_infra2_optical_frame
- added link camera_head_link, mass 0.072; collision box size=0.02505 0.09 0.025; visual mesh filename=file:///home/darsh/ros2_ws/src/UR3_ROS2_PICK_AND_PLACE/inst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
- added link torso_link, mass 2.5; collision box size=0.15 0.10 0.06; collision cylinder length=0.6 radius=0.005
- link base_link_inertia: mass 4.0 -> 2.0; geometry collision mesh filename=package://ur_description/meshes/ur3/collision/base.stl; visual mesh filename=package://ur_description/meshes/ur3/visual/base.dae
- link forearm_link: mass 2.33 -> 1.26; geometry collision mesh filename=package://ur_description/meshes/ur3/collision/forearm.stl; visual mesh filename=package://ur_description/meshes/ur3/visual/forearm.dae
- link shoulder_link: mass 3.7 -> 2.0; geometry collision mesh filename=package://ur_description/meshes/ur3/collision/shoulder.stl; visual mesh filename=package://ur_description/meshes/ur3/visual/shoulder.dae
- link upper_arm_link: mass 8.393 -> 3.42; geometry collision mesh filename=package://ur_description/meshes/ur3/collision/upperarm.stl; visual mesh filename=package://ur_description/meshes/ur3/visual/upperarm.dae
- link wrist_1_link: mass 1.219 -> 0.8; geometry collision mesh filename=package://ur_description/meshes/ur3/collision/wrist1.stl; visual mesh filename=package://ur_description/meshes/ur3/visual/wrist1.dae
- link wrist_2_link: mass 1.219 -> 0.8; geometry collision mesh filename=package://ur_description/meshes/ur3/collision/wrist2.stl; visual mesh filename=package://ur_description/meshes/ur3/visual/wrist2.dae
- link wrist_3_link: mass 0.1879 -> 0.35; geometry collision mesh filename=package://ur_description/meshes/ur3/collision/wrist3.stl; visual mesh filename=package://ur_description/meshes/ur3/visual/wrist3.dae
Joints:
- added joint base_link_to_torso_link: type fixed, parent base_link, child torso_link, origin xyz=0.22 -0.30 0 rpy=0 0 0
- added joint camera_head_color_joint: type fixed, parent camera_head_link, child camera_head_color_frame, origin xyz=0 0.015 0 rpy=0 0 0
- added joint camera_head_color_optical_joint: type fixed, parent camera_head_color_frame, child camera_head_color_optical_frame, origin xyz=0 0 0 rpy=-1.5707963267948966 0 -1.5707963267948966
- added joint camera_head_depth_joint: type fixed, parent camera_head_link, child camera_head_depth_frame, origin xyz=0 0 0 rpy=0 0 0
- added joint camera_head_depth_optical_joint: type fixed, parent camera_head_depth_frame, child camera_head_depth_optical_frame, origin xyz=0 0 0 rpy=-1.5707963267948966 0 -1.5707963267948966
- added joint camera_head_infra1_joint: type fixed, parent camera_head_link, child camera_head_infra1_frame, origin xyz=0 0.0 0 rpy=0 0 0
- added joint camera_head_infra1_optical_joint: type fixed, parent camera_head_infra1_frame, child camera_head_infra1_optical_frame, origin xyz=0 0 0 rpy=-1.5707963267948966 0 -1.5707963267948966
- added joint camera_head_infra2_joint: type fixed, parent camera_head_link, child camera_head_infra2_frame, origin xyz=0 -0.05 0 rpy=0 0 0
- added joint camera_head_infra2_optical_joint: type fixed, parent camera_head_infra2_frame, child camera_head_infra2_optical_frame, origin xyz=0 0 0 rpy=-1.5707963267948966 0 -1.5707963267948966
- added joint camera_head_joint: type fixed, parent torso_link, child camera_head_link, origin xyz=0 0.01 0.50 rpy=0.0 0.4363323129985824 1.5707963267948966
- joint elbow_joint: limit lower=-3.141592653589793 upper=3.141592653589793 effort=150.0 velocity=3.141592653589793 -> lower=-3.141592653589793 upper=3.141592653589793 effort=28.0 velocity=3.141592653589793; origin xyz=-0.425 0 0 rpy=0 0 0 -> xyz=-0.24365 0 0 rpy=0 0 0
- joint shoulder_lift_joint: limit lower=-6.283185307179586 upper=6.283185307179586 effort=150.0 velocity=3.141592653589793 -> lower=-6.283185307179586 upper=6.283185307179586 effort=56.0 velocity=3.141592653589793
- joint shoulder_pan_joint: limit lower=-6.283185307179586 upper=6.283185307179586 effort=150.0 velocity=3.141592653589793 -> lower=-6.283185307179586 upper=6.283185307179586 effort=56.0 velocity=3.141592653589793; origin xyz=0 0 0.089159 rpy=0 0 0 -> xyz=0 0 0.1519 rpy=0 0 0
- joint wrist_1_joint: limit lower=-6.283185307179586 upper=6.283185307179586 effort=28.0 velocity=3.141592653589793 -> lower=-6.283185307179586 upper=6.283185307179586 effort=12.0 velocity=6.283185307179586; origin xyz=-0.39225 0 0.10915 rpy=0 0 0 -> xyz=-0.21325 0 0.11235 rpy=0 0 0
- joint wrist_2_joint: limit lower=-6.283185307179586 upper=6.283185307179586 effort=28.0 velocity=3.141592653589793 -> lower=-6.283185307179586 upper=6.283185307179586 effort=12.0 velocity=6.283185307179586; origin xyz=0 -0.09465 -1.941303950897609e-11 rpy=1.570796327 0 0 -> xyz=0 -0.08535 -1.750557762378351e-11 rpy=1.570796327 0 0
- joint wrist_3_joint: limit lower=-6.283185307179586 upper=6.283185307179586 effort=28.0 velocity=3.141592653589793 -> effort=12.0 velocity=6.283185307179586; origin xyz=0 0.0823 -1.688001216681175e-11 rpy=1.570796326589793 3.141592653589793 3.141592653589793 -> xyz=0 0.0819 -1.679797079540562e-11 rpy=1.570796326589793 3.141592653589793 3.141592653589793; type revolute -> continuous

File: ur_description/urdf/ur.urdf.xacro (robot description, xacro)
@@ -1,13 +1,8 @@
 <?xml version="1.0"?>
 <robot xmlns:xacro="http://wiki.ros.org/xacro" name="$(arg name)">
-   <!-- robot name parameter -->
+   <!-- Declare arguments at the top -->
    <xacro:arg name="name" default="ur"/>
-   <!-- import main macro -->
-   <xacro:include filename="$(find ur_description)/urdf/ur_macro.xacro"/>
-   <!-- possible 'ur_type' values: ur3, ur3e, ur5, ur5e, ur10, ur10e, ur16e, ur20, ur30 -->
-   <!-- the default value should raise an error in case this was called without defining the type -->
-   <xacro:arg name="ur_type" default="ur5"/>
-   <!-- parameters -->
-   <xacro:arg name="tf_prefix" default="" />
+   <xacro:arg name="ur_type" default="ur3"/>
+   <xacro:arg name="tf_prefix" default=""/>
    <xacro:arg name="joint_limit_params" default="$(find ur_description)/config/$(arg ur_type)/joint_limits.yaml"/>
    <xacro:arg name="kinematics_params" default="$(find ur_description)/config/$(arg ur_type)/default_kinematics.yaml"/>
@@ -18,9 +13,10 @@
    <xacro:arg name="safety_pos_margin" default="0.15"/>
    <xacro:arg name="safety_k_position" default="20"/>
-   <!--When using gazebo simulations absolute paths are necessary.-->
-   <xacro:arg name="force_abs_paths" default="false" />
-   <!-- create link fixed to the "world" -->
+   <xacro:arg name="force_abs_paths" default="false"/>
+   <!-- Include main macro after declaring arguments -->
+   <xacro:include filename="$(find ur_description)/urdf/ur_macro.xacro"/>
+   <!-- Create link fixed to the "world" -->
    <link name="world" />
-   <!-- arm -->
+   <!-- Arm -->
    <xacro:ur_robot
      name="$(arg name)"
@@ -34,7 +30,8 @@
      safety_pos_margin="$(arg safety_pos_margin)"
      safety_k_position="$(arg safety_k_position)"
-     force_abs_paths="$(arg force_abs_paths)"
-     >
-     <origin xyz="0 0 0" rpy="0 0 0" />          <!-- position robot in the world -->
+     force_abs_paths="$(arg force_abs_paths)">
+     <origin xyz="0 0 0" rpy="0 0 0" /> <!-- Position robot in the world -->
    </xacro:ur_robot>
+   <!-- Include Intel RealSense Camera -->
+   <xacro:include filename="$(find ur_description)/urdf/intel_rgbd_cam_d435.urdf.xacro"/>
 </robot>
