Commit message: WIP

File: moveit_config/config/ur.urdf (robot description, URDF)
Before this commit: robot ur, 34 links, 33 joints
Joints:
- joint gripper_joint: parent wrist_3_link -> tool0

File: robotiq_2f_85_gripper_visualization/urdf/robotiq_arg2f_85_model_macro.xacro (robot description, xacro)
@@ -2,4 +2,5 @@
 <robot xmlns:xacro="http://ros.org/wiki/xacro">
   <xacro:include filename="$(find robotiq_2f_85_gripper_visualization)/urdf/robotiq_arg2f_transmission.xacro" />
+<xacro:include filename="$(find robotiq_2f_85_gripper_visualization)/urdf/robotiq_arg2f.gazebo.xacro" />
   <xacro:macro name="outer_knuckle" params="prefix fingerprefix stroke">
     <link name="${prefix}${fingerprefix}_outer_knuckle">
@@ -188,4 +189,5 @@
     <xacro:right_outer_knuckle_joint prefix="${prefix}"/>
     <xacro:robotiq_arg2f_transmission prefix="${prefix}"/>
+        <xacro:robotiq_arg2f_gazebo prefix="${prefix}"/>
   </xacro:macro>
 </robot>

File: ur_description/urdf/ur.urdf (robot description, URDF)
Before this commit: robot ur, 34 links, 33 joints
Joints:
- joint gripper_joint: parent wrist_3_link -> tool0

File: ur_description/urdf/ur_macro.xacro (robot description, xacro)
@@ -342,7 +342,7 @@
 <!-- Attach gripper to wrist_3_link with corrected rotation -->
 <joint name="${tf_prefix}gripper_joint" type="fixed">
-  <parent link="${tf_prefix}wrist_3_link"/>
+  <parent link="${tf_prefix}tool0"/>
   <child link="${tf_prefix}robotiq_arg2f_base_link"/>
-  <origin xyz="0 0 0.005" rpy="0 0 ${pi}"/>
+  <origin xyz="0 0 0.005" rpy="0 0 0"/>
 </joint>
 <!-- Define the gripper with a meaningful prefix -->

Commit message: re working config

File: moveit_config/config/ur.urdf (robot description, URDF)
Before this commit: robot ur, 34 links, 33 joints
Links:
- link robotiq_arg2f_base_link: geometry collision mesh filename=package://robotiq_2f_85_gripper_visualization/meshes/visual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 scale=0.001 0.001 0.001; visual mesh filename=package://robotiq_2f_85_gripper_visualization/meshes/visual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 scale=0.001 0.001 0.001
Joints:
- joint right_outer_knuckle_joint: mimic joint=finger_joint multiplier=-1 offset=0 -> joint=finger_joint multiplier=1 offset=0
