Commit message: wip

File: moveit_config/config/ur.ros2_control.xacro (robot description, xacro)
@@ -6,5 +6,4 @@
             <hardware>
                 <!-- By default, set up controllers for simulation. This won't work on real hardware -->
-                <!-- <plugin>mock_components/GenericSystem</plugin> -->
                     <plugin>gz_ros2_control/GazeboSimSystem</plugin>
             </hardware>
@@ -14,6 +13,5 @@
                   <param name="initial_value">${initial_positions['shoulder_pan_joint']}</param>
                 </state_interface>
-                <state_interface name="velocity"/>
-            </joint>
+                           </joint>
             <joint name="shoulder_lift_joint">
                 <command_interface name="position"/>
@@ -21,6 +19,5 @@
                   <param name="initial_value">${initial_positions['shoulder_lift_joint']}</param>
                 </state_interface>
-                <state_interface name="velocity"/>
-            </joint>
+                           </joint>
             <joint name="elbow_joint">
                 <command_interface name="position"/>
@@ -28,5 +25,4 @@
                   <param name="initial_value">${initial_positions['elbow_joint']}</param>
                 </state_interface>
-                <state_interface name="velocity"/>
             </joint>
             <joint name="wrist_1_joint">
@@ -35,5 +31,4 @@
                   <param name="initial_value">${initial_positions['wrist_1_joint']}</param>
                 </state_interface>
-                <state_interface name="velocity"/>
             </joint>
             <joint name="wrist_2_joint">
@@ -42,5 +37,4 @@
                   <param name="initial_value">${initial_positions['wrist_2_joint']}</param>
                 </state_interface>
-                <state_interface name="velocity"/>
             </joint>
             <joint name="wrist_3_joint">
@@ -49,5 +43,4 @@
                   <param name="initial_value">${initial_positions['wrist_3_joint']}</param>
                 </state_interface>
-                <state_interface name="velocity"/>
             </joint>
             <joint name="finger_joint">
@@ -56,6 +49,5 @@
                   <param name="initial_value">${initial_positions['finger_joint']}</param>
                 </state_interface>
-                <state_interface name="velocity"/>
-            </joint>
+                  </joint>
         </ros2_control>
     </xacro:macro>

File: moveit_config/config/ur.urdf.xacro (robot description, xacro)
@@ -8,5 +8,5 @@
     <!-- Import control_xacro -->
     <xacro:include filename="$(find moveit_config)/config/ur.ros2_control.xacro" />
-    <xacro:ur_ros2_control name="FakeSystem" initial_positions_file="$(find ur_description)/config/initial_positions.yaml"/>
+    <xacro:ur_ros2_control name="ur" initial_positions_file="$(find moveit_config)/config/initial_positions.yaml"/>
     <xacro:include filename="$(find ur_description)/urdf/gazebo_sim_ros2_control.urdf.xacro" />
    <xacro:load_gazebo_sim_ros2_control_plugin

File: robotiq_2f_85_gripper_visualization/urdf/robotiq_arg2f.gazebo.xacro (robot description, xacro)
@@ -3,5 +3,5 @@
     <xacro:macro name="robotiq_arg2f_gazebo" params="prefix">
         <gazebo>
-            <plugin filename="libroboticsgroup_gazebo_mimic_joint_plugin.so" name="${prefix}mimic_robotiq_140_1">
+            <plugin filename="libroboticsgroup_gazebo_mimic_joint_plugin.so" name="${prefix}mimic_robotiq_85_1">
                 <joint>${prefix}finger_joint</joint>
                 <mimicJoint>${prefix}right_outer_knuckle_joint</mimicJoint>
@@ -9,5 +9,5 @@
                 <offset>0.0</offset>
             </plugin>
-            <plugin filename="libroboticsgroup_gazebo_mimic_joint_plugin.so" name="${prefix}mimic_robotiq_140_2">
+            <plugin filename="libroboticsgroup_gazebo_mimic_joint_plugin.so" name="${prefix}mimic_robotiq_85_2">
                 <joint>${prefix}finger_joint</joint>
                 <mimicJoint>${prefix}left_inner_knuckle_joint</mimicJoint>
@@ -15,5 +15,5 @@
                 <offset>0.0</offset>
             </plugin>
-            <plugin filename="libroboticsgroup_gazebo_mimic_joint_plugin.so" name="${prefix}mimic_robotiq_140_3">
+            <plugin filename="libroboticsgroup_gazebo_mimic_joint_plugin.so" name="${prefix}mimic_robotiq_85_3">
                 <joint>${prefix}finger_joint</joint>
                 <mimicJoint>${prefix}right_inner_knuckle_joint</mimicJoint>
@@ -21,5 +21,5 @@
                 <offset>0.0</offset>
             </plugin>
-            <plugin filename="libroboticsgroup_gazebo_mimic_joint_plugin.so" name="${prefix}mimic_robotiq_140_4">
+            <plugin filename="libroboticsgroup_gazebo_mimic_joint_plugin.so" name="${prefix}mimic_robotiq_85_4">
                 <joint>${prefix}finger_joint</joint>
                 <mimicJoint>${prefix}left_inner_finger_joint</mimicJoint>
@@ -27,5 +27,5 @@
                 <offset>0.0</offset>
             </plugin>
-            <plugin filename="libroboticsgroup_gazebo_mimic_joint_plugin.so" name="${prefix}mimic_robotiq_140_5">
+            <plugin filename="libroboticsgroup_gazebo_mimic_joint_plugin.so" name="${prefix}mimic_robotiq_85_5">
                 <joint>${prefix}finger_joint</joint>
                 <mimicJoint>${prefix}right_inner_finger_joint</mimicJoint>

File: robotiq_2f_85_gripper_visualization/urdf/robotiq_arg2f.xacro (robot description, xacro)
@@ -20,5 +20,5 @@
         <origin xyz="0 0 0" rpy="0 0 0" />
         <geometry>
-           <mesh filename="package://robotiq_2f_85_gripper_visualization/meshes/collision/robotiq_arg2f_base_link.stl" />
+           <mesh filename="package://robotiq_2f_85_gripper_visualization/meshes/collision/robotiq_arg2f_85_base_link.stl" />
         </geometry>
       </collision>

File: robotiq_2f_85_gripper_visualization/urdf/robotiq_arg2f_85_model_macro.xacro (robot description, xacro)
@@ -177,5 +177,5 @@
       <axis xyz="1 0 0" />
       <limit lower="0" upper="0.81" velocity="2.0" effort="1000" />
-      <mimic joint="${prefix}finger_joint" multiplier="1" offset="0" />
+      <mimic joint="${prefix}finger_joint" multiplier="-1" offset="0" />
     </joint>
     <xacro:finger_joints prefix="${prefix}" fingerprefix="right" reflect="-1.0"/>
@@ -213,6 +213,6 @@
     <xacro:right_outer_knuckle_joint prefix="${prefix}"/>
         <!-- <xacro:left_outer_knuckle_joint prefix="${prefix}"/> -->
-    <xacro:robotiq_arg2f_transmission prefix="${prefix}"/>
-    =<xacro:robotiq_arg2f_gazebo prefix="${prefix}"/>
+    <xacro:robotiq_85_gripper_transmission prefix="${prefix}"/>
+    <xacro:robotiq_arg2f_gazebo prefix="${prefix}"/>
   </xacro:macro>
 </robot>

File: robotiq_2f_85_gripper_visualization/urdf/robotiq_arg2f_transmission.xacro (robot description, xacro)
@@ -1,14 +1,44 @@
 <?xml version="1.0"?>
-<robot xmlns:xacro="http://ros.org/wiki/xacro">
-  <xacro:macro name="robotiq_arg2f_transmission" params="prefix">
-    <transmission name="${prefix}finger_joint_trans">
+<robot xmlns:xacro="http://www.ros.org/wiki/xacro">
+  <xacro:macro name="robotiq_85_gripper_transmission" params="prefix">
+    <transmission name="${prefix}robotiq_85_left_knuckle_trans">
       <type>transmission_interface/SimpleTransmission</type>
-      <joint name="${prefix}finger_joint">
+      <joint name="${prefix}robotiq_85_left_knuckle_joint">
         <hardwareInterface>PositionJointInterface</hardwareInterface>
+        <!-- <hardwareInterface>EffortJointInterface</hardwareInterface> -->
       </joint>
-      <actuator name="${prefix}finger_joint_motor">
+      <actuator name="${prefix}robotiq_85_left_knuckle_motor">
         <mechanicalReduction>1</mechanicalReduction>
+        <hardwareInterface>PositionJointInterface</hardwareInterface>
+        <!-- <hardwareInterface>EfforJointInterface</hardwareInterface> -->
       </actuator>
     </transmission>
+    <!-- Mimic joints -->
+    <gazebo>
+      <plugin filename="libgazebo_mimic_joint_plugin.so" name="${prefix}mimic_robotiq_85_1">
+        <joint>${prefix}robotiq_85_left_knuckle_joint</joint>
+        <mimicJoint>${prefix}robotiq_85_right_knuckle_joint</mimicJoint>
+      </plugin>
+      <plugin filename="libgazebo_mimic_joint_plugin.so" name="${prefix}mimic_robotiq_85_2">
+        <joint>${prefix}robotiq_85_left_knuckle_joint</joint>
+        <mimicJoint>${prefix}robotiq_85_left_inner_knuckle_joint</mimicJoint>
+      </plugin>
+      <plugin filename="libgazebo_mimic_joint_plugin.so" name="${prefix}mimic_robotiq_85_3">
+        <joint>${prefix}robotiq_85_left_knuckle_joint</joint>
+        <mimicJoint>${prefix}robotiq_85_right_inner_knuckle_joint</mimicJoint>
+      </plugin>
+      <plugin filename="libgazebo_mimic_joint_plugin.so" name="${prefix}mimic_robotiq_85_4">
+        <joint>${prefix}robotiq_85_left_knuckle_joint</joint>
+        <mimicJoint>${prefix}robotiq_85_left_finger_tip_joint</mimicJoint>
+        <multiplier>-1.0</multiplier>
+        <offset>0.0</offset>
+      </plugin>
+      <plugin filename="libgazebo_mimic_joint_plugin.so" name="${prefix}mimic_robotiq_85_5">
+        <joint>${prefix}robotiq_85_left_knuckle_joint</joint>
+        <mimicJoint>${prefix}robotiq_85_right_finger_tip_joint</mimicJoint>
+        <multiplier>-1.0</multiplier>
+        <offset>0.0</offset>
+      </plugin>
+    </gazebo>
   </xacro:macro>
 </robot>

File: ur_description/urdf/gazebo_sim_ros2_control.urdf.xacro (robot description, xacro)
@@ -6,9 +6,7 @@
                 <plugin filename="gz_ros2_control-system" name="gz_ros2_control::GazeboSimROS2ControlPlugin">
                     <parameters>$(find moveit_config)/config/ros2_controllers.yaml</parameters>
-                    <!-- Uncomment this if controller_manager has issues finding robot_description -->
                     <ros>
                         <remapping>/controller_manager/robot_description:=/robot_description</remapping>
                     </ros>
-                    <controller_manager_node_name>controller_manager</controller_manager_node_name>
                 </plugin>
             </gazebo>

File: ur_description/urdf/ur.urdf.xacro (robot description, xacro)
@@ -1,4 +1,4 @@
 <?xml version="1.0"?>
-<robot xmlns:xacro="http://wiki.ros.org/xacro" name="$(arg name)">
+<robot xmlns:xacro="http://wiki.ros.org/xacro" name="ur">
    <!-- Declare arguments at the top -->
    <xacro:arg name="name" default="ur"/>
@@ -35,12 +35,11 @@
      <origin xyz="0 0 0" rpy="0 0 0" /> <!-- Position robot in the world -->
    </xacro:ur_robot>
-   <!-- Include Gazebo Simulation Control Plugin -->
-   <xacro:include filename="$(find ur_description)/urdf/gazebo_sim_ros2_control.urdf.xacro" />
+<!--
+=   <xacro:include filename="$(find ur_description)/urdf/gazebo_sim_ros2_control.urdf.xacro" />
    <xacro:load_gazebo_sim_ros2_control_plugin
      robot_name="$(arg robot_name)"
      use_gazebo="$(arg use_gazebo)"/>
-   <!-- UR-Specific ROS 2 Control -->
    <xacro:include filename="$(find ur_description)/urdf/ur.ros2_control.xacro" />
-<xacro:ur_ros2_control name="ur_robot" initial_positions_file="$(find ur_description)/config/initial_positions.yaml"/>
+<xacro:ur_ros2_control name="ur_robot" initial_positions_file="$(find ur_description)/config/initial_positions.yaml"/> -->
    <!-- Include Intel RealSense Camera -->
    <xacro:include filename="$(find ur_description)/urdf/intel_rgbd_cam_d435.urdf.xacro"/>

File: ur_description/urdf/ur_macro.xacro (robot description, xacro)
@@ -304,10 +304,10 @@
       <dynamics damping="0" friction="0"/>
     </joint>
-    <!-- <link name="${tf_prefix}ft_frame"/>
+    <link name="${tf_prefix}ft_frame"/>
     <joint name="${tf_prefix}wrist_3_link-ft_frame" type="fixed">
       <parent link="${tf_prefix}wrist_3_link"/>
       <child link="${tf_prefix}ft_frame"/>
       <origin xyz="0 0 0" rpy="${pi} 0 0"/>
-    </joint> -->
+    </joint>
     <!-- ROS-Industrial 'base' frame - base_link to UR 'Base' Coordinates transform -->
    <link name="${tf_prefix}base"/>
@@ -322,5 +322,4 @@
   <child link="${tf_prefix}base"/>
   </joint>
-  <!-- ROS-Industrial 'flange' frame - attachment point for EEF models
   <link name="${tf_prefix}flange" />
   <joint name="${tf_prefix}wrist_3-flange" type="fixed">
@@ -328,13 +327,11 @@
   <child link="${tf_prefix}flange" />
   <origin xyz="0 0 0" rpy="0 ${-pi/2.0} ${-pi/2.0}" />
-  </joint> -->
-  <!-- ROS-Industrial 'tool0' frame - all-zeros tool frame -->
-  <!-- <link name="${tf_prefix}tool0"/>
-  <joint name="${tf_prefix}flange-tool0" type="fixed"> -->
-  <!-- default toolframe - X+ left, Y+ up, Z+ front -->
-  <!-- <origin xyz="0 0 0" rpy="${pi/2.0} 0 ${pi/2.0}"/>
+  </joint>
+  <link name="${tf_prefix}tool0"/>
+  <joint name="${tf_prefix}flange-tool0" type="fixed">
+  <origin xyz="0 0 0" rpy="${pi/2.0} 0 ${pi/2.0}"/>
   <parent link="${tf_prefix}flange"/>
   <child link="${tf_prefix}tool0"/>
-  </joint> -->
+  </joint>
    <xacro:include filename="$(find robotiq_2f_85_gripper_visualization)/urdf/robotiq_arg2f_85_model_macro.xacro"/>
   <!-- Include the gripper Xacro file  -->
@@ -343,5 +340,5 @@
 <!-- Attach gripper to wrist_3_link with corrected rotation -->
 <joint name="${tf_prefix}gripper_joint" type="fixed">
-  <parent link="${tf_prefix}wrist_3_link"/>
+  <parent link="${tf_prefix}tool0"/>
   <child link="${tf_prefix}robotiq_arg2f_base_link"/>
   <origin xyz="0 0 0.005" rpy="0 0 0"/>

File: ur_robot.urdf (robot description, URDF)
Before this commit: robot ur, 34 links, 33 joints
Joints:
- joint gripper_joint: type fixed -> revolute

Commit message: controlling arm gazebo

File: moveit_config/config/ur.ros2_control.xacro (robot description, xacro)
@@ -49,4 +49,5 @@
                   <param name="initial_value">${initial_positions['finger_joint']}</param>
                 </state_interface>
+                    <!-- <state_interface name="velocity"/>  🔥 This is the missing piece -->
                   </joint>
         </ros2_control>

File: moveit_config/config/ur.urdf.xacro (robot description, xacro)
@@ -5,5 +5,5 @@
    <xacro:arg name="robot_name" default="ur"/>
     <!-- Import ur urdf file -->
-    <xacro:include filename="$(find ur_description)/urdf/ur.urdf" />
+    <xacro:include filename="$(find ur_description)/urdf/ur.urdf.xacro" />
     <!-- Import control_xacro -->
     <xacro:include filename="$(find moveit_config)/config/ur.ros2_control.xacro" />

File: robotiq_2f_85_gripper_visualization/urdf/robotiq_arg2f_85_model_macro.xacro (robot description, xacro)
@@ -2,5 +2,5 @@
 <robot xmlns:xacro="http://ros.org/wiki/xacro">
   <xacro:include filename="$(find robotiq_2f_85_gripper_visualization)/urdf/robotiq_arg2f_transmission.xacro" />
-<xacro:include filename="$(find robotiq_2f_85_gripper_visualization)/urdf/robotiq_arg2f.gazebo.xacro" />
+<!-- <xacro:include filename="$(find robotiq_2f_85_gripper_visualization)/urdf/robotiq_arg2f.gazebo.xacro" /> -->
   <xacro:include filename="$(find robotiq_2f_85_gripper_visualization)/urdf/robotiq_arg2f.xacro" />
   <xacro:macro name="outer_knuckle" params="prefix fingerprefix stroke">
@@ -149,5 +149,5 @@
       <axis xyz="1 0 0" />
       <limit lower="-0.8757" upper="0" velocity="2.0" effort="1000" />
-      <mimic joint="${prefix}finger_joint" multiplier="-1" offset="0" />
+      <mimic joint="${prefix}finger_joint" multiplier="1" offset="0" />
     </joint>
   </xacro:macro>
@@ -207,12 +207,21 @@
   <!-- Initialization of all joints and links -->
   <xacro:macro name="robotiq_arg2f_85" params="prefix">
-    <xacro:robotiq_arg2f_base_link prefix="${prefix}"/>
+      <xacro:robotiq_arg2f_base_link prefix="${prefix}"/>
     <xacro:finger_links prefix="${prefix}" fingerprefix="left" stroke="85"/>
     <xacro:finger_links prefix="${prefix}" fingerprefix="right" stroke="85"/>
-    <xacro:finger_joint prefix="${prefix}"/>
+   <xacro:finger_joints prefix="${prefix}" fingerprefix="left" reflect="1.0"/>
+    <xacro:finger_joints prefix="${prefix}" fingerprefix="right" reflect="-1.0"/>
     <xacro:right_outer_knuckle_joint prefix="${prefix}"/>
         <!-- <xacro:left_outer_knuckle_joint prefix="${prefix}"/> -->
     <xacro:robotiq_85_gripper_transmission prefix="${prefix}"/>
-    <xacro:robotiq_arg2f_gazebo prefix="${prefix}"/>
+    <!-- <xacro:robotiq_arg2f_gazebo prefix="${prefix}"/> -->
+ <gazebo reference="${prefix}robotiq_arg2f_base_link">
+      <physics>
+        <ode>
+          <implicit_spring_damper>1</implicit_spring_damper>
+          <cfm_damping_reference_velocity>0.01</cfm_damping_reference_velocity>
+        </ode>
+      </physics>
+    </gazebo>
   </xacro:macro>
 </robot>

File: robotiq_2f_85_gripper_visualization/urdf/robotiq_arg2f_transmission.xacro (robot description, xacro)
@@ -2,18 +2,28 @@
 <robot xmlns:xacro="http://www.ros.org/wiki/xacro">
   <xacro:macro name="robotiq_85_gripper_transmission" params="prefix">
-    <transmission name="${prefix}robotiq_85_left_knuckle_trans">
+    <!-- <transmission name="${prefix}robotiq_85_left_knuckle_trans">
       <type>transmission_interface/SimpleTransmission</type>
       <joint name="${prefix}robotiq_85_left_knuckle_joint">
         <hardwareInterface>PositionJointInterface</hardwareInterface>
-        <!-- <hardwareInterface>EffortJointInterface</hardwareInterface> -->
+        <hardwareInterface>EffortJointInterface</hardwareInterface>
       </joint>
       <actuator name="${prefix}robotiq_85_left_knuckle_motor">
         <mechanicalReduction>1</mechanicalReduction>
         <hardwareInterface>PositionJointInterface</hardwareInterface>
-        <!-- <hardwareInterface>EfforJointInterface</hardwareInterface> -->
+        <hardwareInterface>EfforJointInterface</hardwareInterface>
       </actuator>
-    </transmission>
+    </transmission> -->
+    <transmission name="${prefix}robotiq_85_finger_joint_trans">
+  <type>transmission_interface/SimpleTransmission</type>
+  <joint name="${prefix}finger_joint">
+    <hardwareInterface>PositionJointInterface</hardwareInterface>
+  </joint>
+  <actuator name="${prefix}finger_motor">
+    <hardwareInterface>PositionJointInterface</hardwareInterface>
+    <mechanicalReduction>1</mechanicalReduction>
+  </actuator>
+</transmission>
     <!-- Mimic joints -->
-    <gazebo>
+    <!-- <gazebo>
       <plugin filename="libgazebo_mimic_joint_plugin.so" name="${prefix}mimic_robotiq_85_1">
         <joint>${prefix}robotiq_85_left_knuckle_joint</joint>
@@ -40,5 +50,5 @@
         <offset>0.0</offset>
       </plugin>
-    </gazebo>
+    </gazebo> -->
   </xacro:macro>
 </robot>

File: ur_description/urdf/gazebo_sim_ros2_control.urdf.xacro (robot description, xacro)
@@ -4,5 +4,5 @@
         <xacro:if value="${use_gazebo}">
             <gazebo>
-                <plugin filename="gz_ros2_control-system" name="gz_ros2_control::GazeboSimROS2ControlPlugin">
+<plugin name="gz_ros2_control" filename="libgz_ros2_control-system.so">
                     <parameters>$(find moveit_config)/config/ros2_controllers.yaml</parameters>
                     <ros>

File: ur_description/urdf/ur.urdf (robot description, URDF)
Before this commit: robot ur, 34 links, 33 joints
Joints:
- removed joint finger_joint
- removed joint right_outer_knuckle_joint

File: ur_description/urdf/ur_macro.xacro (robot description, xacro)
@@ -336,5 +336,5 @@
    <xacro:include filename="$(find robotiq_2f_85_gripper_visualization)/urdf/robotiq_arg2f_85_model_macro.xacro"/>
   <!-- Include the gripper Xacro file  -->
-<xacro:robotiq_arg2f_85 prefix="$(arg tf_prefix)"/>
+<xacro:robotiq_arg2f_85 prefix=""/>
 <!-- Attach the gripper to tool0 -->
 <!-- Attach gripper to wrist_3_link with corrected rotation -->

Commit message: fixed mimic joint

File: moveit_config/config/ur.ros2_control.xacro (robot description, xacro)
@@ -57,4 +57,40 @@
                 <state_interface name="velocity"/>
             </joint>
+            <!-- Mimic joints (no command interfaces, initial value same as finger_joint) -->
+<!-- right_outer_knuckle_joint -->
+<joint name="right_outer_knuckle_joint">
+  <state_interface name="position">
+    <param name="initial_value">${initial_positions['finger_joint']}</param>
+  </state_interface>
+  <state_interface name="velocity"/>
+</joint>
+<!-- right_inner_knuckle_joint -->
+<joint name="right_inner_knuckle_joint">
+  <state_interface name="position">
+    <param name="initial_value">${initial_positions['finger_joint']}</param>
+  </state_interface>
+  <state_interface name="velocity"/>
+</joint>
+<!-- left_inner_knuckle_joint -->
+<joint name="left_inner_knuckle_joint">
+  <state_interface name="position">
+    <param name="initial_value">${initial_positions['finger_joint']}</param>
+  </state_interface>
+  <state_interface name="velocity"/>
+</joint>
+<!-- right_inner_finger_joint -->
+<joint name="right_inner_finger_joint">
+  <state_interface name="position">
+    <param name="initial_value">${initial_positions['finger_joint']}</param>
+  </state_interface>
+  <state_interface name="velocity"/>
+</joint>
+<!-- left_inner_finger_joint -->
+<joint name="left_inner_finger_joint">
+  <state_interface name="position">
+    <param name="initial_value">${initial_positions['finger_joint']}</param>
+  </state_interface>
+  <state_interface name="velocity"/>
+</joint>
         </ros2_control>
     </xacro:macro>
