Commit message: gazwbo fix

File: moveit_config/config/ur.urdf.xacro (robot description, xacro)
@@ -8,4 +8,7 @@
     <!-- Import control_xacro -->
     <xacro:include filename="$(find moveit_config)/config/ur.ros2_control.xacro" />
+    <gazebo>
+  <disableFixedJointLumping>true</disableFixedJointLumping>
+</gazebo>
     <xacro:ur_ros2_control name="ur" initial_positions_file="$(find moveit_config)/config/initial_positions.yaml"/>
     <xacro:include filename="$(find ur_description)/urdf/gazebo_sim_ros2_control.urdf.xacro" />

File: robotiq_2f_85_gripper_visualization/urdf/robotiq_arg2f.xacro (robot description, xacro)
@@ -11,5 +11,5 @@
         <origin xyz="0 0 0" rpy="0 0 0" />
         <geometry>
-          <mesh filename="package://robotiq_2f_85_gripper_visualization/meshes/visual/robotiq_arg2f_85_base_link.dae" scale="0.001 0.001 0.001"/>
+          <mesh filename="package://robotiq_2f_85_gripper_visualization/meshes/collision/robotiq_arg2f_85_base_link.stl"/>
         </geometry>
         <material name="">
@@ -20,8 +20,11 @@
         <origin xyz="0 0 0" rpy="0 0 0" />
         <geometry>
-           <mesh filename="package://robotiq_2f_85_gripper_visualization/meshes/collision/robotiq_arg2f_base_link.stl" />
+          <mesh filename="package://robotiq_2f_85_gripper_visualization/meshes/collision/robotiq_arg2f_85_base_link.stl" />
         </geometry>
       </collision>
     </link>
+    <gazebo reference="robotiq_arg2f_base_link">
+  <disableFixedJointLumping>true</disableFixedJointLumping>
+</gazebo>
   </xacro:macro>
   <xacro:macro name="finger_joints" params="prefix fingerprefix reflect">

File: robotiq_2f_85_gripper_visualization/urdf/robotiq_arg2f_85_model_macro.xacro (robot description, xacro)
@@ -188,4 +188,7 @@
     <xacro:right_outer_knuckle_joint prefix="${prefix}"/>
     <xacro:robotiq_arg2f_transmission prefix="${prefix}"/>
+    <gazebo>
+  <disableFixedJointLumping>true</disableFixedJointLumping>
+</gazebo>
   </xacro:macro>
 </robot>

File: ur_description/urdf/ur_macro.xacro (robot description, xacro)
@@ -343,4 +343,7 @@
   <child link="${tf_prefix}robotiq_arg2f_base_link"/>
   <origin xyz="0 0 0.005" rpy="0 0 0"/>
+    <gazebo>
+    <disableFixedJointLumping>true</disableFixedJointLumping>
+  </gazebo>
 </joint>
 <!-- Define the gripper with a meaningful prefix -->
