Commit message: increased controller delay loading time

File: robotiq_2f_85_gripper_visualization/urdf/robotiq_arg2f_85_model_macro.xacro (robot description, xacro)
@@ -102,5 +102,5 @@
     <link name="${prefix}${fingerprefix}_inner_finger_pad">
       <visual>
-        <origin xyz="0 0 0" rpy="0 0 0" />
+        <origin xyz="0 0 0" rpy="0 0 0" />f
         <geometry>
           <box size="0.022 0.00635 0.0375"/>
