Commit message: minor change:

File: robotiq_2f_85_gripper_visualization/urdf/robotiq_arg2f.xacro (robot description, xacro)
@@ -20,5 +20,5 @@
         <origin xyz="0 0 0" rpy="0 0 0" />
         <geometry>
-           <mesh filename="package://robotiq_2f_85_gripper_visualization/meshes/collision/robotiq_arg2f_85_base_link.stl" />
+           <mesh filename="package://robotiq_2f_85_gripper_visualization/meshes/collision/robotiq_arg2f_base_link.stl" />
         </geometry>
       </collision>

File: robotiq_2f_85_gripper_visualization/urdf/robotiq_arg2f_85_model_macro.xacro (robot description, xacro)
@@ -2,6 +2,4 @@
 <robot xmlns:xacro="http://ros.org/wiki/xacro">
   <xacro:include filename="$(find robotiq_2f_85_gripper_visualization)/urdf/robotiq_arg2f_transmission.xacro" />
-<!-- <xacro:include filename="$(find robotiq_2f_85_gripper_visualization)/urdf/robotiq_arg2f.gazebo.xacro" /> -->
-  <xacro:include filename="$(find robotiq_2f_85_gripper_visualization)/urdf/robotiq_arg2f.xacro" />
   <xacro:macro name="outer_knuckle" params="prefix fingerprefix stroke">
     <link name="${prefix}${fingerprefix}_outer_knuckle">
@@ -160,4 +158,5 @@
     </joint>
   </xacro:macro>
+  <xacro:include filename="$(find robotiq_2f_85_gripper_visualization)/urdf/robotiq_arg2f.xacro" />
   <xacro:macro name="finger_joint" params="prefix">
     <joint name="${prefix}finger_joint" type="revolute">
@@ -181,48 +180,12 @@
     <xacro:finger_joints prefix="${prefix}" fingerprefix="right" reflect="-1.0"/>
   </xacro:macro>
-  <xacro:macro name="robotiq_arg2f_base_link" params="prefix">
-    <link name="${prefix}robotiq_arg2f_base_link">
-      <inertial>
-        <origin xyz="8.625E-08 -4.6583E-06 0.03145" rpy="0 0 0" />
-        <mass value="0.22652" />
-        <inertia ixx="0.00020005" ixy="-4.2442E-10" ixz="-2.9069E-10" iyy="0.00017832" iyz="-3.4402E-08" izz="0.00013478" />
-      </inertial>
-      <visual>
-        <origin xyz="0 0 0" rpy="0 0 0" />
-        <geometry>
-          <mesh filename="package://robotiq_2f_85_gripper_visualization/meshes/visual/robotiq_arg2f_85_base_link.dae" scale="0.001 0.001 0.001"/>
-        </geometry>
-        <material name="">
-          <color rgba="0.1 0.1 0.1 1" />
-        </material>
-      </visual>
-      <collision>
-        <origin xyz="0 0 0" rpy="0 0 0" />
-        <geometry>
-          <mesh filename="package://robotiq_2f_85_gripper_visualization/meshes/visual/robotiq_arg2f_85_base_link.dae" scale="0.001 0.001 0.001"/>
-        </geometry>
-      </collision>
-    </link>
-  </xacro:macro>
   <!-- Initialization of all joints and links -->
   <xacro:macro name="robotiq_arg2f_85" params="prefix">
-      <xacro:robotiq_arg2f_base_link prefix="${prefix}"/>
-          <xacro:finger_joint prefix="${prefix}"/>
+    <xacro:robotiq_arg2f_base_link prefix="${prefix}"/>
     <xacro:finger_links prefix="${prefix}" fingerprefix="left" stroke="85"/>
     <xacro:finger_links prefix="${prefix}" fingerprefix="right" stroke="85"/>
-   <!-- <xacro:finger_joints prefix="${prefix}" fingerprefix="left" reflect="1.0"/> -->
-    <!-- <xacro:finger_joints prefix="${prefix}" fingerprefix="right" reflect="-1.0"/>  -->
+    <xacro:finger_joint prefix="${prefix}"/>
     <xacro:right_outer_knuckle_joint prefix="${prefix}"/>
-        <!-- <xacro:left_outer_knuckle_joint prefix="${prefix}"/> -->
-    <xacro:robotiq_85_gripper_transmission prefix="${prefix}"/>
-    <!-- <xacro:robotiq_arg2f_gazebo prefix="${prefix}"/> -->
- <gazebo reference="${prefix}robotiq_arg2f_base_link">
-      <physics>
-        <ode>
-          <implicit_spring_damper>1</implicit_spring_damper>
-          <cfm_damping_reference_velocity>0.01</cfm_damping_reference_velocity>
-        </ode>
-      </physics>
-    </gazebo>
+    <xacro:robotiq_arg2f_transmission prefix="${prefix}"/>
   </xacro:macro>
 </robot>

File: robotiq_2f_85_gripper_visualization/urdf/robotiq_arg2f_transmission.xacro (robot description, xacro)
@@ -1,54 +1,14 @@
 <?xml version="1.0"?>
-<robot xmlns:xacro="http://www.ros.org/wiki/xacro">
-  <xacro:macro name="robotiq_85_gripper_transmission" params="prefix">
-    <!-- <transmission name="${prefix}robotiq_85_left_knuckle_trans">
+<robot xmlns:xacro="http://ros.org/wiki/xacro">
+  <xacro:macro name="robotiq_arg2f_transmission" params="prefix">
+    <transmission name="${prefix}finger_joint_trans">
       <type>transmission_interface/SimpleTransmission</type>
-      <joint name="${prefix}robotiq_85_left_knuckle_joint">
+      <joint name="${prefix}finger_joint">
         <hardwareInterface>PositionJointInterface</hardwareInterface>
-        <hardwareInterface>EffortJointInterface</hardwareInterface>
       </joint>
-      <actuator name="${prefix}robotiq_85_left_knuckle_motor">
+      <actuator name="${prefix}finger_joint_motor">
         <mechanicalReduction>1</mechanicalReduction>
-        <hardwareInterface>PositionJointInterface</hardwareInterface>
-        <hardwareInterface>EfforJointInterface</hardwareInterface>
       </actuator>
-    </transmission> -->
-    <transmission name="${prefix}robotiq_85_finger_joint_trans">
-  <type>transmission_interface/SimpleTransmission</type>
-  <joint name="${prefix}finger_joint">
-    <hardwareInterface>PositionJointInterface</hardwareInterface>
-  </joint>
-  <actuator name="${prefix}finger_motor">
-    <hardwareInterface>PositionJointInterface</hardwareInterface>
-    <mechanicalReduction>1</mechanicalReduction>
-  </actuator>
-</transmission>
-    <!-- Mimic joints -->
-    <!-- <gazebo>
-      <plugin filename="libgazebo_mimic_joint_plugin.so" name="${prefix}mimic_robotiq_85_1">
-        <joint>${prefix}robotiq_85_left_knuckle_joint</joint>
-        <mimicJoint>${prefix}robotiq_85_right_knuckle_joint</mimicJoint>
-      </plugin>
-      <plugin filename="libgazebo_mimic_joint_plugin.so" name="${prefix}mimic_robotiq_85_2">
-        <joint>${prefix}robotiq_85_left_knuckle_joint</joint>
-        <mimicJoint>${prefix}robotiq_85_left_inner_knuckle_joint</mimicJoint>
-      </plugin>
-      <plugin filename="libgazebo_mimic_joint_plugin.so" name="${prefix}mimic_robotiq_85_3">
-        <joint>${prefix}robotiq_85_left_knuckle_joint</joint>
-        <mimicJoint>${prefix}robotiq_85_right_inner_knuckle_joint</mimicJoint>
-      </plugin>
-      <plugin filename="libgazebo_mimic_joint_plugin.so" name="${prefix}mimic_robotiq_85_4">
-        <joint>${prefix}robotiq_85_left_knuckle_joint</joint>
-        <mimicJoint>${prefix}robotiq_85_left_finger_tip_joint</mimicJoint>
-        <multiplier>-1.0</multiplier>
-        <offset>0.0</offset>
-      </plugin>
-      <plugin filename="libgazebo_mimic_joint_plugin.so" name="${prefix}mimic_robotiq_85_5">
-        <joint>${prefix}robotiq_85_left_knuckle_joint</joint>
-        <mimicJoint>${prefix}robotiq_85_right_finger_tip_joint</mimicJoint>
-        <multiplier>-1.0</multiplier>
-        <offset>0.0</offset>
-      </plugin>
-    </gazebo> -->
+    </transmission>
   </xacro:macro>
 </robot>

File: ur_description/urdf/gazebo_sim_ros2_control.urdf.xacro (robot description, xacro)
@@ -4,5 +4,5 @@
         <xacro:if value="${use_gazebo}">
             <gazebo>
-<plugin name="gz_ros2_control" filename="libgz_ros2_control-system.so">
+                <plugin filename="gz_ros2_control-system" name="gz_ros2_control::GazeboSimROS2ControlPlugin">
                     <parameters>$(find moveit_config)/config/ros2_controllers.yaml</parameters>
                     <ros>

Commit message: minor changes

File: robotiq_2f_85_gripper_visualization/urdf/robotiq_arg2f.xacro (robot description, xacro)
@@ -20,5 +20,5 @@
         <origin xyz="0 0 0" rpy="0 0 0" />
         <geometry>
-          <mesh filename="package://robotiq_2f_85_gripper_visualization/meshes/collision/robotiq_arg2f_85_base_link.stl" />
+          <mesh filename="package://robotiq_2f_85_gripper_visualization/meshes/collision/robotiq_arg2f_85_base_link.stl"/>
         </geometry>
       </collision>

File: ur_description/urdf/ur.urdf (robot description, URDF)
Before this commit: robot ur, 34 links, 33 joints
Links:
- link robotiq_arg2f_base_link: geometry collision mesh filename=package://robotiq_2f_85_gripper_visualization/meshes/collis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 scale=0.001 0.001 0.001; visual mesh filename=package://robotiq_2f_85_gripper_visualization/meshes/collis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
Joints:
- joint left_inner_finger_joint: mimic joint=finger_joint multiplier=1 offset=0 -> joint=finger_joint multiplier=-1 offset=0
- joint right_inner_finger_joint: mimic joint=finger_joint multiplier=1 offset=0 -> joint=finger_joint multiplier=-1 offset=0
- joint right_outer_knuckle_joint: mimic joint=finger_joint multiplier=-1 offset=0 -> joint=finger_joint multiplier=1 offset=0
