Commit message: fixing pick error

File: install/robotiq_2f_85_gripper_visualization/share/robotiq_2f_85_gripper_visualization/urdf/robotiq_arg2f.xacro (robot description, xacro)
@@ -1,43 +1 @@
-<?xml version="1.0"?>
-<robot xmlns:xacro="http://ros.org/wiki/xacro">
-  <xacro:macro name="robotiq_arg2f_base_link" params="prefix">
-    <link name="${prefix}robotiq_arg2f_base_link">
-      <inertial>
-        <origin xyz="8.625E-08 -4.6583E-06 0.03145" rpy="0 0 0" />
-        <mass value="0.22652" />
-        <inertia ixx="0.00020005" ixy="-4.2442E-10" ixz="-2.9069E-10" iyy="0.00017832" iyz="-3.4402E-08" izz="0.00013478" />
-      </inertial>
-      <visual>
-        <origin xyz="0 0 0" rpy="0 0 0" />
-        <geometry>
-          <mesh filename="package://robotiq_2f_85_gripper_visualization/meshes/collision/robotiq_arg2f_85_base_link.stl"/>
-        </geometry>
-        <material name="">
-          <color rgba="0.1 0.1 0.1 1" />
-        </material>
-      </visual>
-      <!-- <collision>
-        <origin xyz="0 0 0" rpy="0 0 0" />
-        <geometry>
-          <mesh filename="package://robotiq_2f_85_gripper_visualization/meshes/collision/robotiq_arg2f_85_base_link.stl"/>
-        </geometry>
-      </collision> -->
-    </link>
-    <gazebo reference="robotiq_arg2f_base_link">
-  <disableFixedJointLumping>true</disableFixedJointLumping>
-</gazebo>
-  </xacro:macro>
-  <xacro:macro name="finger_joints" params="prefix fingerprefix reflect">
-    <xacro:outer_finger_joint prefix="${prefix}" fingerprefix="${fingerprefix}"/>
-    <xacro:inner_knuckle_joint prefix="${prefix}" fingerprefix="${fingerprefix}" reflect="${reflect}"/>
-    <xacro:inner_finger_joint prefix="${prefix}" fingerprefix="${fingerprefix}"/>
-    <xacro:inner_finger_pad_joint prefix="${prefix}" fingerprefix="${fingerprefix}"/>
-  </xacro:macro>
-  <xacro:macro name="finger_links" params="prefix fingerprefix stroke">
-    <xacro:outer_knuckle prefix="${prefix}" fingerprefix="${fingerprefix}" stroke="${stroke}"/>
-    <xacro:outer_finger prefix="${prefix}" fingerprefix="${fingerprefix}" stroke="${stroke}"/>
-    <xacro:inner_finger prefix="${prefix}" fingerprefix="${fingerprefix}" stroke="${stroke}"/>
-    <xacro:inner_finger_pad prefix="${prefix}" fingerprefix="${fingerprefix}"/>
-    <xacro:inner_knuckle prefix="${prefix}" fingerprefix="${fingerprefix}" stroke="${stroke}"/>
-  </xacro:macro>
-</robot>
+/home/darsh/UR3_ROS2_PICK_AND_PLACE/robotiq_2f_85_gripper_visualization/urdf/robotiq_arg2f.xacro

File: install/robotiq_2f_85_gripper_visualization/share/robotiq_2f_85_gripper_visualization/urdf/robotiq_arg2f_85_model_macro.xacro (robot description, xacro)
@@ -1,194 +1 @@
-<?xml version="1.0"?>
-<robot xmlns:xacro="http://ros.org/wiki/xacro">
-  <xacro:include filename="$(find robotiq_2f_85_gripper_visualization)/urdf/robotiq_arg2f_transmission.xacro" />
-  <xacro:macro name="outer_knuckle" params="prefix fingerprefix stroke">
-    <link name="${prefix}${fingerprefix}_outer_knuckle">
-      <inertial>
-        <origin xyz="-0.000200000000003065 0.0199435877845359 0.0292245259211331" rpy="0 0 0" />
-        <mass value="0.00853198276973456" />
-        <inertia ixx="2.89328108496468E-06" ixy="-1.57935047237397E-19" ixz="-1.93980378593255E-19" iyy="1.86719750325683E-06" iyz="-1.21858577871576E-06" izz="1.21905238907251E-06" />
-        </inertial>
-      <visual>
-        <origin xyz="0 0 0" rpy="0 0 0" />
-        <geometry>
-          <mesh filename="package://robotiq_2f_85_gripper_visualization/meshes/visual/robotiq_arg2f_85_outer_knuckle.dae" scale="0.001 0.001 0.001"/>
-        </geometry>
-        <material name="">
-          <color rgba="0.792156862745098 0.819607843137255 0.933333333333333 1" />
-        </material>
-      </visual>
-      <collision>
-        <origin xyz="0 0 0" rpy="0 0 0" />
-        <geometry>
-          <mesh filename="package://robotiq_2f_85_gripper_visualization/meshes/collision/robotiq_arg2f_85_outer_knuckle.dae" scale="0.001 0.001 0.001"/>
-        </geometry>
-      </collision>
-    </link>
-  </xacro:macro>
-  <xacro:macro name="outer_finger" params="prefix fingerprefix stroke">
-    <link name="${prefix}${fingerprefix}_outer_finger">
-      <inertial>
-        <origin xyz="0.00030115855001899 0.0373907951953854 -0.0208027427000385" rpy="0 0 0" />
-        <mass value="0.022614240507152" />
-        <inertia ixx="1.52518312458174E-05" ixy="9.76583423954399E-10" ixz="-5.43838577022588E-10" iyy="6.17694243867776E-06" iyz="6.78636130740228E-06" izz="1.16494917907219E-05" />
-        </inertial>
-      <visual>
-        <origin xyz="0 0 0" rpy="0 0 0" />
-        <geometry>
-          <mesh filename="package://robotiq_2f_85_gripper_visualization/meshes/visual/robotiq_arg2f_85_outer_finger.dae" scale="0.001 0.001 0.001"/>
-        </geometry>
-        <material name="">
-          <color rgba="0.1 0.1 0.1 1" />
-        </material>
-      </visual>
-      <collision>
-        <origin xyz="0 0 0" rpy="0 0 0" />
-        <geometry>
-          <mesh filename="package://robotiq_2f_85_gripper_visualization/meshes/collision/robotiq_arg2f_85_outer_finger.dae" scale="0.001 0.001 0.001"/>
-        </geometry>
-      </collision>
-    </link>
-  </xacro:macro>
-  <xacro:macro name="inner_knuckle" params="prefix fingerprefix stroke">
-    <link name="${prefix}${fingerprefix}_inner_knuckle">
-      <inertial>
-        <origin xyz="0.000123011831763771 0.0507850843201817 0.00103968640075166" rpy="0 0 0" />
-       <mass value="0.0271177346495152" />
-        <inertia ixx="2.61910379223783E-05" ixy="-2.43616858946494E-07" ixz="-6.37789906117123E-09" iyy="2.8270243746167E-06" iyz="-5.37200748039765E-07" izz="2.83695868220296E-05" />
-        </inertial>
-      <visual>
-        <origin xyz="0 0 0" rpy="0 0 0" />
-        <geometry>
-          <mesh filename="package://robotiq_2f_85_gripper_visualization/meshes/visual/robotiq_arg2f_85_inner_knuckle.dae" scale="0.001 0.001 0.001"/>
-        </geometry>
-        <material name="">
-          <color rgba="0.1 0.1 0.1 1" />
-        </material>
-      </visual>
-      <collision>
-        <origin xyz="0 0 0" rpy="0 0 0" />
-        <geometry>
-          <mesh filename="package://robotiq_2f_85_gripper_visualization/meshes/collision/robotiq_arg2f_85_inner_knuckle.dae" scale="0.001 0.001 0.001"/>
-        </geometry>
-      </collision>
-    </link>
-  </xacro:macro>
-  <xacro:macro name="inner_finger" params="prefix fingerprefix stroke">
-    <link name="${prefix}${fingerprefix}_inner_finger">
-      <inertial>
-        <origin xyz="0.000299999999999317 0.0160078233491243 -0.0136945669206257" rpy="0 0 0" />
-        <mass value="0.0104003125914103" />
-        <inertia ixx="2.71909453810972E-06" ixy="1.35402465472579E-21" ixz="-7.1817349065269E-22" iyy="7.69100314106116E-07" iyz="6.74715432769696E-07" izz="2.30315190420171E-06" />
-        </inertial>
-      <visual>
-        <origin xyz="0 0 0" rpy="0 0 0" />
-        <geometry>
-          <mesh filename="package://robotiq_2f_85_gripper_visualization/meshes/visual/robotiq_arg2f_85_inner_finger.dae" scale="0.001 0.001 0.001"/>
-        </geometry>
-        <material name="">
-          <color rgba="0.1 0.1 0.1 1" />
-        </material>
-      </visual>
-      <collision>
-        <origin xyz="0 0 0" rpy="0 0 0" />
-        <geometry>
-          <mesh filename="package://robotiq_2f_85_gripper_visualization/meshes/collision/robotiq_arg2f_85_inner_finger.dae" scale="0.001 0.001 0.001" />
-        </geometry>
-      </collision>
-    </link>
-  </xacro:macro>
-   <!-- Finger pad link, the default are the "big pads" with rubber-->
-  <xacro:macro name="inner_finger_pad" params="prefix fingerprefix">
-    <link name="${prefix}${fingerprefix}_inner_finger_pad">
-      <visual>
-        <origin xyz="0 0 0" rpy="0 0 0" />f
-        <geometry>
-          <box size="0.022 0.00635 0.0375"/>
-        </geometry>
-        <material name="">
-          <color rgba="0.9 0.9 0.9 1" />
-        </material>
-      </visual>
-      <collision>
-        <origin xyz="0 0 0" rpy="0 0 0" />
-        <geometry>
-           <box size="0.022 0.00635 0.0375"/>
-        </geometry>
-        <material name="">
-          <color rgba="0.9 0.0 0.0 1" />
-        </material>
-      </collision>
-    </link>
-  </xacro:macro>
-  <xacro:macro name="outer_finger_joint" params="prefix fingerprefix">
-    <joint name="${prefix}${fingerprefix}_outer_finger_joint" type="fixed">
-      <origin xyz="0 0.0315 -0.0041" rpy="0 0 0"/>
-      <parent link="${prefix}${fingerprefix}_outer_knuckle" />
-      <child link="${prefix}${fingerprefix}_outer_finger" />
-      <axis xyz="1 0 0" />
-    </joint>
-  </xacro:macro>
-  <xacro:macro name="inner_knuckle_joint" params="prefix fingerprefix reflect">
-    <joint name="${prefix}${fingerprefix}_inner_knuckle_joint" type="revolute">
-      <!-- <origin xyz="0 ${reflect * -0.0127} 0.06142" rpy="${pi / 2 + .725} 0 ${(reflect - 1) * pi / 2}" /> -->
-      <origin xyz="0 ${reflect * -0.0127} 0.06142" rpy="0 0 ${(1 + reflect) * pi / 2}"/>
-      <parent link="${prefix}robotiq_arg2f_base_link" />
-      <child link="${prefix}${fingerprefix}_inner_knuckle" />
-      <axis xyz="1 0 0" />
-      <limit lower="0" upper="0.8757" velocity="2.0" effort="1000" />
-      <mimic joint="${prefix}finger_joint" multiplier="1" offset="0" />
-    </joint>
-  </xacro:macro>
-  <xacro:macro name="inner_finger_joint" params="prefix fingerprefix">
-    <joint name="${prefix}${fingerprefix}_inner_finger_joint" type="revolute">
-      <origin xyz="0 0.0061 0.0471" rpy="0 0 0"/>
-      <parent link="${prefix}${fingerprefix}_outer_finger" />
-      <child link="${prefix}${fingerprefix}_inner_finger" />
-      <axis xyz="1 0 0" />
-      <limit lower="-0.8757" upper="0" velocity="2.0" effort="1000" />
-      <mimic joint="${prefix}finger_joint" multiplier="-1" offset="0" />
-    </joint>
-  </xacro:macro>
-  <xacro:macro name="inner_finger_pad_joint" params="prefix fingerprefix">
-    <joint name="${prefix}${fingerprefix}_inner_finger_pad_joint" type="fixed">
-      <origin xyz="0 -0.0220203446692936 0.03242" rpy="0 0 0"/>
-      <parent link="${prefix}${fingerprefix}_inner_finger" />
-      <child link="${prefix}${fingerprefix}_inner_finger_pad" />
-      <axis xyz="0 0 1" />
-    </joint>
-  </xacro:macro>
-  <xacro:include filename="$(find robotiq_2f_85_gripper_visualization)/urdf/robotiq_arg2f.xacro" />
-  <xacro:macro name="finger_joint" params="prefix">
-    <joint name="${prefix}finger_joint" type="revolute">
-      <origin xyz="0 -0.0306011 0.054904" rpy="0 0 ${pi}"/>
-      <parent link="${prefix}robotiq_arg2f_base_link" />
-      <child link="${prefix}left_outer_knuckle" />
-      <axis xyz="1 0 0" />
-      <limit lower="0" upper="0.8" velocity="2.0" effort="1000" />
-    </joint>
-    <xacro:finger_joints prefix="${prefix}" fingerprefix="left" reflect="1.0"/>
-  </xacro:macro>
-  <xacro:macro name="right_outer_knuckle_joint" params="prefix">
-    <joint name="${prefix}right_outer_knuckle_joint" type="revolute">
-      <origin xyz="0 0.0306011 0.054904" rpy="0 0 0"/>
-      <parent link="${prefix}robotiq_arg2f_base_link" />
-      <child link="${prefix}right_outer_knuckle" />
-      <axis xyz="1 0 0" />
-      <limit lower="0" upper="0.81" velocity="2.0" effort="1000" />
-      <mimic joint="${prefix}finger_joint" multiplier="1" offset="0" />
-    </joint>
-    <xacro:finger_joints prefix="${prefix}" fingerprefix="right" reflect="-1.0"/>
-  </xacro:macro>
-  <!-- Initialization of all joints and links -->
-  <xacro:macro name="robotiq_arg2f_85" params="prefix">
-    <xacro:robotiq_arg2f_base_link prefix="${prefix}"/>
-    <xacro:finger_links prefix="${prefix}" fingerprefix="left" stroke="85"/>
-    <xacro:finger_links prefix="${prefix}" fingerprefix="right" stroke="85"/>
-    <xacro:finger_joint prefix="${prefix}"/>
-    <xacro:right_outer_knuckle_joint prefix="${prefix}"/>
-    <xacro:robotiq_arg2f_transmission prefix="${prefix}"/>
-    <gazebo>
-  <disableFixedJointLumping>true</disableFixedJointLumping>
-</gazebo>
-  </xacro:macro>
-</robot>
+/home/darsh/UR3_ROS2_PICK_AND_PLACE/robotiq_2f_85_gripper_visualization/urdf/robotiq_arg2f_85_model_macro.xacro

File: install/robotiq_2f_85_gripper_visualization/share/robotiq_2f_85_gripper_visualization/urdf/robotiq_arg2f_transmission.xacro (robot description, xacro)
@@ -1,14 +1 @@
-<?xml version="1.0"?>
-<robot xmlns:xacro="http://ros.org/wiki/xacro">
-  <xacro:macro name="robotiq_arg2f_transmission" params="prefix">
-    <transmission name="${prefix}finger_joint_trans">
-      <type>transmission_interface/SimpleTransmission</type>
-      <joint name="${prefix}finger_joint">
-        <hardwareInterface>PositionJointInterface</hardwareInterface>
-      </joint>
-      <actuator name="${prefix}finger_joint_motor">
-        <mechanicalReduction>1</mechanicalReduction>
-      </actuator>
-    </transmission>
-  </xacro:macro>
-</robot>
+/home/darsh/UR3_ROS2_PICK_AND_PLACE/robotiq_2f_85_gripper_visualization/urdf/robotiq_arg2f_transmission.xacro

File: install/ur_description/share/ur_description/urdf/gazebo_sim_ros2_control.urdf.xacro (robot description, xacro)
@@ -1,15 +1 @@
-<?xml version="1.0" ?>
-<robot xmlns:xacro="http://wiki.ros.org/xacro">
-    <xacro:macro name="load_gazebo_sim_ros2_control_plugin" params="robot_name use_gazebo">
-        <xacro:if value="${use_gazebo}">
-            <gazebo>
-                <plugin filename="gz_ros2_control-system" name="gz_ros2_control::GazeboSimROS2ControlPlugin">
-                    <parameters>$(find moveit_config)/config/ros2_controllers.yaml</parameters>
-                    <ros>
-                        <remapping>/controller_manager/robot_description:=/robot_description</remapping>
-                    </ros>
-                </plugin>
-            </gazebo>
-        </xacro:if>
-    </xacro:macro>
-</robot>
+/home/darsh/UR3_ROS2_PICK_AND_PLACE/ur_description/urdf/gazebo_sim_ros2_control.urdf.xacro

File: install/ur_description/share/ur_description/urdf/intel_rgbd_cam_d435.urdf.xacro (robot description, xacro)
@@ -1,157 +1 @@
-<?xml version="1.0"?>
-<robot xmlns:xacro="http://www.ros.org/wiki/xacro">
-  <xacro:arg name="use_camera" default="true"/>
-  <xacro:arg name="use_gazebo" default="true"/>
-  <xacro:arg name="prefix" default=""/>
-  <xacro:if value="${'true' == '$(arg use_camera)' and 'true' == '$(arg use_gazebo)'}">
-    <xacro:property name="M_PI" value="3.1415926535897931" />
-    <xacro:property name="d435_cam_width" value="0.090"/>
-    <xacro:property name="d435_cam_height" value="0.025"/>
-    <xacro:property name="d435_cam_depth" value="0.02505"/>
-    <xacro:property name="d435_cam_depth_to_infra1_offset" value="0.0"/>
-    <xacro:property name="d435_cam_depth_to_infra2_offset" value="-0.050"/>
-    <xacro:property name="d435_cam_depth_to_color_offset" value="0.015"/>
-    <xacro:property name="camera_tilt_angle_deg" value="25"/>
-    <link name="torso_link">
-      <inertial>
-        <origin xyz="0 0 0.50" />
-        <mass value="2.5" />
-        <inertia ixx="0.8" ixy="0.0" ixz="0.0" iyy="0.8" iyz="0.0" izz="0.8" />
-      </inertial>
-      <visual name="holder">
-        <origin xyz="0 0 0.25" rpy="0 0 0" />
-        <material name="LightGrey">
-          <color rgba="0.7 0.7 0.7 1.0"/>
-        </material>
-        <geometry>
-          <cylinder radius="0.005" length="0.5"/>
-        </geometry>
-      </visual>
-      <visual name="base">
-        <origin xyz="0 0 0" rpy="0 0 0" />
-        <material name="LightGrey">
-          <color rgba="0.7 0.7 0.7 1.0"/>
-        </material>
-        <geometry>
-          <box size="0.15 0.10 0.06" />
-        </geometry>
-      </visual>
-      <collision name="holder">
-        <origin xyz="0 0 0.25" rpy="0 0 0" />
-        <geometry>
-          <cylinder radius="0.005" length="0.6"/>
-        </geometry>
-      </collision>
-      <collision name="base">
-        <origin xyz="0 0 0.0" rpy="0 0 0" />
-        <geometry>
-          <box size="0.15 0.10 0.06" />
-        </geometry>
-      </collision>
-    </link>
-    <joint name="$(arg prefix)base_link_to_torso_link" type="fixed">
-      <parent link="$(arg prefix)base_link"/>
-      <child link="torso_link"/>
-      <origin xyz="0.22 -0.30 0" rpy="0 0 0"/>
-    </joint>
-    <joint name="camera_head_joint" type="fixed">
-      <parent link="torso_link"/>
-      <child link="camera_head_link" />
-      <origin xyz="0 0.01 0.50" rpy="0.0 ${camera_tilt_angle_deg * M_PI / 180} ${M_PI/2}"/>
-    </joint>
-    <link name="camera_head_link">
-      <visual>
-        <origin xyz="0 0 0" rpy="${M_PI/2} 0.0 ${M_PI/2}"/>
-        <geometry>
-          <mesh filename="file://$(find ur_description)/meshes/d435/visual/d435.stl" />
-        </geometry>
-        <material name="aluminum">
-          <color rgba="0.5 0.5 0.5 1"/>
-        </material>
-      </visual>
-      <collision>
-        <origin xyz="0 0 0" rpy="0 0 0"/>
-        <geometry>
-          <box size="${d435_cam_depth} ${d435_cam_width} ${d435_cam_height}"/>
-        </geometry>
-      </collision>
-      <inertial>
-        <mass value="0.072" />
-        <origin xyz="0 0 0" />
-        <inertia ixx="0.003881243" ixy="0.0" ixz="0.0" iyy="0.000498940" iyz="0.0" izz="0.003879257" />
-      </inertial>
-    </link>
-    <joint name="camera_head_depth_joint" type="fixed">
-      <origin xyz="0 0 0" rpy="0 0 0"/>
-      <parent link="camera_head_link"/>
-      <child link="camera_head_depth_frame" />
-    </joint>
-    <link name="camera_head_depth_frame"/>
-    <joint name="camera_head_depth_optical_joint" type="fixed">
-      <origin xyz="0 0 0" rpy="${-M_PI/2} 0 ${-M_PI/2}" />
-      <parent link="camera_head_depth_frame" />
-      <child link="camera_head_depth_optical_frame" />
-    </joint>
-    <link name="camera_head_depth_optical_frame"/>
-    <joint name="camera_head_infra1_joint" type="fixed">
-      <origin xyz="0 ${d435_cam_depth_to_infra1_offset} 0" rpy="0 0 0" />
-      <parent link="camera_head_link" />
-      <child link="camera_head_infra1_frame" />
-    </joint>
-    <link name="camera_head_infra1_frame"/>
-    <joint name="camera_head_infra1_optical_joint" type="fixed">
-      <origin xyz="0 0 0" rpy="${-M_PI/2} 0 ${-M_PI/2}" />
-      <parent link="camera_head_infra1_frame" />
-      <child link="camera_head_infra1_optical_frame" />
-    </joint>
-    <link name="camera_head_infra1_optical_frame"/>
-    <joint name="camera_head_infra2_joint" type="fixed">
-      <origin xyz="0 ${d435_cam_depth_to_infra2_offset} 0" rpy="0 0 0" />
-      <parent link="camera_head_link" />
-      <child link="camera_head_infra2_frame" />
-    </joint>
-    <link name="camera_head_infra2_frame"/>
-    <joint name="camera_head_infra2_optical_joint" type="fixed">
-      <origin xyz="0 0 0" rpy="${-M_PI/2} 0 ${-M_PI/2}" />
-      <parent link="camera_head_infra2_frame" />
-      <child link="camera_head_infra2_optical_frame" />
-    </joint>
-    <link name="camera_head_infra2_optical_frame"/>
-    <joint name="camera_head_color_joint" type="fixed">
-      <origin xyz="0 ${d435_cam_depth_to_color_offset} 0" rpy="0 0 0" />
-      <parent link="camera_head_link" />
-      <child link="camera_head_color_frame" />
-    </joint>
-    <link name="camera_head_color_frame"/>
-    <joint name="camera_head_color_optical_joint" type="fixed">
-      <origin xyz="0 0 0" rpy="${-M_PI/2} 0 ${-M_PI/2}" />
-      <parent link="camera_head_color_frame" />
-      <child link="camera_head_color_optical_frame" />
-    </joint>
-    <link name="camera_head_color_optical_frame"/>
-<gazebo reference="camera_head_link">
-  <sensor name="camera_head" type="rgbd_camera">
-    <camera>
-      <horizontal_fov>1.5184</horizontal_fov>
-      <image>
-        <width>424</width>
-        <height>240</height>
-      </image>
-      <clip>
-        <near>0.05</near>
-        <far>1.5</far>
-      </clip>
-    </camera>
-    <always_on>1</always_on>
-    <update_rate>10</update_rate>
-    <gz_frame_id>camera_head_link</gz_frame_id>
-    <output>
-      <image>true</image>
-      <depth_image>true</depth_image>
-      <point_cloud>true</point_cloud>
-    </output>
-    <visualize>true</visualize>
-  </sensor>
-</gazebo>
-  </xacro:if>
-</robot>
+/home/darsh/UR3_ROS2_PICK_AND_PLACE/ur_description/urdf/intel_rgbd_cam_d435.urdf.xacro

File: install/ur_description/share/ur_description/urdf/ur.urdf.xacro (robot description, xacro)
@@ -1,46 +1 @@
-<?xml version="1.0"?>
-<robot xmlns:xacro="http://wiki.ros.org/xacro" name="ur">
-   <!-- Declare arguments at the top -->
-   <xacro:arg name="name" default="ur"/>
-   <xacro:arg name="ur_type" default="ur3"/>
-   <xacro:arg name="tf_prefix" default=""/>
-   <xacro:arg name="joint_limit_params" default="$(find ur_description)/config/$(arg ur_type)/joint_limits.yaml"/>
-   <xacro:arg name="kinematics_params" default="$(find ur_description)/config/$(arg ur_type)/default_kinematics.yaml"/>
-   <xacro:arg name="physical_params" default="$(find ur_description)/config/$(arg ur_type)/physical_parameters.yaml"/>
-   <xacro:arg name="visual_params" default="$(find ur_description)/config/$(arg ur_type)/visual_parameters.yaml"/>
-   <xacro:arg name="transmission_hw_interface" default=""/>
-   <xacro:arg name="safety_limits" default="false"/>
-   <xacro:arg name="safety_pos_margin" default="0.15"/>
-   <xacro:arg name="safety_k_position" default="20"/>
-   <xacro:arg name="force_abs_paths" default="false"/>
-   <xacro:arg name="robot_name" default="ur"/>
-   <xacro:arg name="use_gazebo" default="true"/> <!-- Added missing argument -->
-   <!-- Include main macro after declaring arguments -->
-   <xacro:include filename="$(find ur_description)/urdf/ur_macro.xacro"/>
-   <!-- Create link fixed to the "world" -->
-   <link name="world" />
-   <!-- Arm -->
-   <xacro:ur_robot
-     name="$(arg name)"
-     tf_prefix="$(arg tf_prefix)"
-     parent="world"
-     joint_limits_parameters_file="$(arg joint_limit_params)"
-     kinematics_parameters_file="$(arg kinematics_params)"
-     physical_parameters_file="$(arg physical_params)"
-     visual_parameters_file="$(arg visual_params)"
-     safety_limits="$(arg safety_limits)"
-     safety_pos_margin="$(arg safety_pos_margin)"
-     safety_k_position="$(arg safety_k_position)"
-     force_abs_paths="$(arg force_abs_paths)">
-     <origin xyz="0 0 0" rpy="0 0 0" /> <!-- Position robot in the world -->
-   </xacro:ur_robot>
-<!--
-=   <xacro:include filename="$(find ur_description)/urdf/gazebo_sim_ros2_control.urdf.xacro" />
-   <xacro:load_gazebo_sim_ros2_control_plugin
-     robot_name="$(arg robot_name)"
-     use_gazebo="$(arg use_gazebo)"/>
-   <xacro:include filename="$(find ur_description)/urdf/ur.ros2_control.xacro" />
-<xacro:ur_ros2_control name="ur_robot" initial_positions_file="$(find ur_description)/config/initial_positions.yaml"/> -->
-   <!-- Include Intel RealSense Camera -->
-   <xacro:include filename="$(find ur_description)/urdf/intel_rgbd_cam_d435.urdf.xacro"/>
-</robot>
+/home/darsh/UR3_ROS2_PICK_AND_PLACE/ur_description/urdf/ur.urdf.xacro
