Commit message: no IK solution WIP

File: install/moveit_config/share/moveit_config/config/ur.urdf (robot description, URDF)
Before this commit: robot ur, 34 links, 33 joints
Links:
- link robotiq_arg2f_base_link: geometry collision mesh filename=package://robotiq_2f_85_gripper_visualization/meshes/collis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; visual mesh filename=package://robotiq_2f_85_gripper_visualization/meshes/visual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 scale=0.001 0.001 0.001

File: install/ur_description/share/ur_description/urdf/ur.urdf (robot description, URDF)
Before this commit: robot ur, 34 links, 33 joints
Links:
- link robotiq_arg2f_base_link: geometry collision mesh filename=package://robotiq_2f_85_gripper_visualization/meshes/collis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 scale=0.001 0.001 0.001; visual mesh filename=package://robotiq_2f_85_gripper_visualization/meshes/collis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
- link torso_link: geometry collision box size=0.15 0.10 0.06; collision cylinder length=0.6 radius=0.005
Joints:
- joint camera_head_joint: origin xyz=0 0.01 0.8 rpy=0.0 0.4363323129985824 1.5707963267948966 -> xyz=0 0.01 0.50 rpy=0.0 0.4363323129985824 1.5707963267948966

Commit message: WIP

File: install/moveit_config/share/moveit_config/config/ur.urdf (robot description, URDF)
Before this commit: robot ur, 34 links, 33 joints
Links:
- link robotiq_arg2f_base_link: geometry collision mesh filename=package://robotiq_2f_85_gripper_visualization/meshes/collis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; visual mesh filename=package://robotiq_2f_85_gripper_visualization/meshes/collis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
Joints:
- joint wrist_3_joint: limit effort=12.0 velocity=6.283185307179586 -> lower=-6.283185307179586 upper=6.283185307179586 effort=12.0 velocity=6.283185307179586; type continuous -> revolute

File: install/ur_description/share/ur_description/urdf/inc/ur_common.xacro (robot description, xacro)
@@ -76,12 +76,12 @@
     <xacro:property name="wrist_2_velocity_limit" value="${sec_limits['wrist_2_joint']['max_velocity']}" scope="parent"/>
     <xacro:property name="wrist_2_effort_limit" value="${sec_limits['wrist_2_joint']['max_effort']}" scope="parent"/>
-    <xacro:if value="${sec_limits['wrist_3_joint']['has_position_limits']}">
+    <!-- <xacro:if value="${sec_limits['wrist_3_joint']['has_position_limits']}"> -->
       <xacro:property name="wrist_3_joint_type" value="revolute" scope="parent"/>
       <xacro:property name="wrist_3_lower_limit" value="${sec_limits['wrist_3_joint']['min_position']}" scope="parent"/>
       <xacro:property name="wrist_3_upper_limit" value="${sec_limits['wrist_3_joint']['max_position']}" scope="parent"/>
-    </xacro:if>
-    <xacro:unless value="${sec_limits['wrist_3_joint']['has_position_limits']}">
+    <!-- </xacro:if> -->
+    <!-- <xacro:unless value="${sec_limits['wrist_3_joint']['has_position_limits']}">
       <xacro:property name="wrist_3_joint_type" value="continuous" scope="parent"/>
-    </xacro:unless>
+    </xacro:unless> -->
     <xacro:property name="wrist_3_velocity_limit" value="${sec_limits['wrist_3_joint']['max_velocity']}" scope="parent"/>
     <xacro:property name="wrist_3_effort_limit" value="${sec_limits['wrist_3_joint']['max_effort']}" scope="parent"/>

File: install/ur_description/share/ur_description/urdf/ur.urdf (robot description, URDF)
Before this commit: robot ur, 34 links, 33 joints
Joints:
- joint wrist_3_joint: type continuous -> revolute

File: install/ur_description/share/ur_description/urdf/ur_macro.xacro (robot description, xacro)
@@ -284,10 +284,10 @@
       <dynamics damping="0" friction="0"/>
     </joint>
-    <joint name="${tf_prefix}wrist_3_joint" type="${wrist_3_joint_type}">
+    <joint name="${tf_prefix}wrist_3_joint" type="revolute">
       <parent link="${tf_prefix}wrist_2_link" />
       <child link="${tf_prefix}wrist_3_link" />
       <origin xyz="${wrist_3_x} ${wrist_3_y} ${wrist_3_z}" rpy="${wrist_3_roll} ${wrist_3_pitch} ${wrist_3_yaw}" />
       <axis xyz="0 0 1" />
-      <xacro:if value="${wrist_3_joint_type != 'continuous'}">
+      <!-- <xacro:if value="${wrist_3_joint_type != 'continuous'}"> -->
         <limit lower="${wrist_3_lower_limit}" upper="${wrist_3_upper_limit}"
           effort="${wrist_3_effort_limit}" velocity="${wrist_3_velocity_limit}"/>
@@ -295,11 +295,11 @@
           <safety_controller soft_lower_limit="${wrist_3_lower_limit + safety_pos_margin}" soft_upper_limit="${wrist_3_upper_limit - safety_pos_margin}" k_position="${safety_k_position}" k_velocity="0.0"/>
         </xacro:if>
-      </xacro:if>
-      <xacro:unless value="${wrist_3_joint_type != 'continuous'}">
+      <!-- </xacro:if> -->
+      <!-- <xacro:unless value="${wrist_3_joint_type != 'continuous'}"> -->
         <limit effort="${wrist_3_effort_limit}" velocity="${wrist_3_velocity_limit}"/>
         <xacro:if value="${safety_limits}">
           <safety_controller k_position="${safety_k_position}" k_velocity="0.0"/>
         </xacro:if>
-      </xacro:unless>
+      <!-- </xacro:unless> -->
       <dynamics damping="0" friction="0"/>
     </joint>

Commit message: reverted change

File: install/moveit_config/share/moveit_config/config/ur.urdf (robot description, URDF)
Before this commit: robot ur, 34 links, 33 joints
Links:
- link robotiq_arg2f_base_link: geometry collision mesh filename=package://robotiq_2f_85_gripper_visualization/meshes/collis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; visual mesh filename=package://robotiq_2f_85_gripper_visualization/meshes/visual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 scale=0.001 0.001 0.001
Joints:
- joint wrist_3_joint: limit lower=-6.283185307179586 upper=6.283185307179586 effort=12.0 velocity=6.283185307179586 -> effort=12.0 velocity=6.283185307179586; type revolute -> continuous

File: install/ur_description/share/ur_description/urdf/inc/ur_common.xacro (robot description, xacro)
@@ -76,12 +76,12 @@
     <xacro:property name="wrist_2_velocity_limit" value="${sec_limits['wrist_2_joint']['max_velocity']}" scope="parent"/>
     <xacro:property name="wrist_2_effort_limit" value="${sec_limits['wrist_2_joint']['max_effort']}" scope="parent"/>
-    <!-- <xacro:if value="${sec_limits['wrist_3_joint']['has_position_limits']}"> -->
+    <xacro:if value="${sec_limits['wrist_3_joint']['has_position_limits']}">
       <xacro:property name="wrist_3_joint_type" value="revolute" scope="parent"/>
       <xacro:property name="wrist_3_lower_limit" value="${sec_limits['wrist_3_joint']['min_position']}" scope="parent"/>
       <xacro:property name="wrist_3_upper_limit" value="${sec_limits['wrist_3_joint']['max_position']}" scope="parent"/>
-    <!-- </xacro:if> -->
-    <!-- <xacro:unless value="${sec_limits['wrist_3_joint']['has_position_limits']}">
+    </xacro:if>
+    <xacro:unless value="${sec_limits['wrist_3_joint']['has_position_limits']}">
       <xacro:property name="wrist_3_joint_type" value="continuous" scope="parent"/>
-    </xacro:unless> -->
+    </xacro:unless>
     <xacro:property name="wrist_3_velocity_limit" value="${sec_limits['wrist_3_joint']['max_velocity']}" scope="parent"/>
     <xacro:property name="wrist_3_effort_limit" value="${sec_limits['wrist_3_joint']['max_effort']}" scope="parent"/>

File: install/ur_description/share/ur_description/urdf/ur.urdf (robot description, URDF)
Before this commit: robot ur, 34 links, 33 joints
Joints:
- joint wrist_3_joint: type revolute -> continuous

File: install/ur_description/share/ur_description/urdf/ur_macro.xacro (robot description, xacro)
@@ -284,10 +284,10 @@
       <dynamics damping="0" friction="0"/>
     </joint>
-    <joint name="${tf_prefix}wrist_3_joint" type="revolute">
+    <joint name="${tf_prefix}wrist_3_joint" type="${wrist_3_joint_type}">
       <parent link="${tf_prefix}wrist_2_link" />
       <child link="${tf_prefix}wrist_3_link" />
       <origin xyz="${wrist_3_x} ${wrist_3_y} ${wrist_3_z}" rpy="${wrist_3_roll} ${wrist_3_pitch} ${wrist_3_yaw}" />
       <axis xyz="0 0 1" />
-      <!-- <xacro:if value="${wrist_3_joint_type != 'continuous'}"> -->
+      <xacro:if value="${wrist_3_joint_type != 'continuous'}">
         <limit lower="${wrist_3_lower_limit}" upper="${wrist_3_upper_limit}"
           effort="${wrist_3_effort_limit}" velocity="${wrist_3_velocity_limit}"/>
@@ -295,11 +295,11 @@
           <safety_controller soft_lower_limit="${wrist_3_lower_limit + safety_pos_margin}" soft_upper_limit="${wrist_3_upper_limit - safety_pos_margin}" k_position="${safety_k_position}" k_velocity="0.0"/>
         </xacro:if>
-      <!-- </xacro:if> -->
-      <!-- <xacro:unless value="${wrist_3_joint_type != 'continuous'}"> -->
+      </xacro:if>
+      <xacro:unless value="${wrist_3_joint_type != 'continuous'}">
         <limit effort="${wrist_3_effort_limit}" velocity="${wrist_3_velocity_limit}"/>
         <xacro:if value="${safety_limits}">
           <safety_controller k_position="${safety_k_position}" k_velocity="0.0"/>
         </xacro:if>
-      <!-- </xacro:unless> -->
+      </xacro:unless>
       <dynamics damping="0" friction="0"/>
     </joint>
