Commit message: added execution

File: install/moveit_config/share/moveit_config/config/ur.ros2_control.xacro (robot description, xacro)
@@ -6,91 +6,127 @@
             <hardware>
                 <!-- By default, set up controllers for simulation. This won't work on real hardware -->
-                    <plugin>gz_ros2_control/GazeboSimSystem</plugin>
+                <plugin>gz_ros2_control/GazeboSimSystem</plugin>
             </hardware>
             <joint name="shoulder_pan_joint">
                 <command_interface name="position"/>
                 <state_interface name="position">
-                  <param name="initial_value">${initial_positions['shoulder_pan_joint']}</param>
+                    <param name="initial_value">${initial_positions['shoulder_pan_joint']}</param>
                 </state_interface>
                 <state_interface name="velocity"/>
+                <state_interface name="effort"> <!-- Adding effort interface -->
+                    <param name="effort_limit">50.0</param> <!-- Torque limit in Nm -->
+                </state_interface>
             </joint>
             <joint name="shoulder_lift_joint">
                 <command_interface name="position"/>
                 <state_interface name="position">
-                  <param name="initial_value">${initial_positions['shoulder_lift_joint']}</param>
+                    <param name="initial_value">${initial_positions['shoulder_lift_joint']}</param>
                 </state_interface>
                 <state_interface name="velocity"/>
+                <state_interface name="effort">
+                    <param name="effort_limit">50.0</param>
+                </state_interface>
             </joint>
             <joint name="elbow_joint">
                 <command_interface name="position"/>
                 <state_interface name="position">
-                  <param name="initial_value">${initial_positions['elbow_joint']}</param>
+                    <param name="initial_value">${initial_positions['elbow_joint']}</param>
                 </state_interface>
                 <state_interface name="velocity"/>
+                <state_interface name="effort">
+                    <param name="effort_limit">50.0</param>
+                </state_interface>
             </joint>
             <joint name="wrist_1_joint">
                 <command_interface name="position"/>
                 <state_interface name="position">
-                  <param name="initial_value">${initial_positions['wrist_1_joint']}</param>
+                    <param name="initial_value">${initial_positions['wrist_1_joint']}</param>
                 </state_interface>
                 <state_interface name="velocity"/>
+                <state_interface name="effort">
+                    <param name="effort_limit">50.0</param>
+                </state_interface>
             </joint>
             <joint name="wrist_2_joint">
                 <command_interface name="position"/>
                 <state_interface name="position">
-                  <param name="initial_value">${initial_positions['wrist_2_joint']}</param>
+                    <param name="initial_value">${initial_positions['wrist_2_joint']}</param>
                 </state_interface>
                 <state_interface name="velocity"/>
+                <state_interface name="effort">
+                    <param name="effort_limit">50.0</param>
+                </state_interface>
             </joint>
             <joint name="wrist_3_joint">
                 <command_interface name="position"/>
                 <state_interface name="position">
-                  <param name="initial_value">${initial_positions['wrist_3_joint']}</param>
+                    <param name="initial_value">${initial_positions['wrist_3_joint']}</param>
                 </state_interface>
                 <state_interface name="velocity"/>
+                <state_interface name="effort">
+                    <param name="effort_limit">50.0</param>
+                </state_interface>
             </joint>
             <joint name="finger_joint">
                 <command_interface name="position"/>
                 <state_interface name="position">
-                  <param name="initial_value">${initial_positions['finger_joint']}</param>
+                    <param name="initial_value">${initial_positions['finger_joint']}</param>
                 </state_interface>
                 <state_interface name="velocity"/>
+                <state_interface name="effort">
+                    <param name="effort_limit">100.0</param> <!-- Increased effort for finger strength -->
+                </state_interface>
             </joint>
             <!-- Mimic joints (no command interfaces, initial value same as finger_joint) -->
-<!-- right_outer_knuckle_joint -->
-<joint name="right_outer_knuckle_joint">
-  <state_interface name="position">
-    <param name="initial_value">${initial_positions['finger_joint']}</param>
-  </state_interface>
-  <state_interface name="velocity"/>
-</joint>
-<!-- right_inner_knuckle_joint -->
-<joint name="right_inner_knuckle_joint">
-  <state_interface name="position">
-    <param name="initial_value">${initial_positions['finger_joint']}</param>
-  </state_interface>
-  <state_interface name="velocity"/>
-</joint>
-<!-- left_inner_knuckle_joint -->
-<joint name="left_inner_knuckle_joint">
-  <state_interface name="position">
-    <param name="initial_value">${initial_positions['finger_joint']}</param>
-  </state_interface>
-  <state_interface name="velocity"/>
-</joint>
-<!-- right_inner_finger_joint -->
-<joint name="right_inner_finger_joint">
-  <state_interface name="position">
-    <param name="initial_value">${initial_positions['finger_joint']}</param>
-  </state_interface>
-  <state_interface name="velocity"/>
-</joint>
-<!-- left_inner_finger_joint -->
-<joint name="left_inner_finger_joint">
-  <state_interface name="position">
-    <param name="initial_value">${initial_positions['finger_joint']}</param>
-  </state_interface>
-  <state_interface name="velocity"/>
-</joint>
+            <!-- right_outer_knuckle_joint -->
+            <joint name="right_outer_knuckle_joint">
+                <state_interface name="position">
+                    <param name="initial_value">${initial_positions['finger_joint']}</param>
+                </state_interface>
+                <state_interface name="velocity"/>
+                <state_interface name="effort">
+                    <param name="effort_limit">100.0</param> <!-- Increased effort for knuckle strength -->
+                </state_interface>
+            </joint>
+            <!-- right_inner_knuckle_joint -->
+            <joint name="right_inner_knuckle_joint">
+                <state_interface name="position">
+                    <param name="initial_value">${initial_positions['finger_joint']}</param>
+                </state_interface>
+                <state_interface name="velocity"/>
+                <state_interface name="effort">
+                    <param name="effort_limit">100.0</param>
+                </state_interface>
+            </joint>
+            <!-- left_inner_knuckle_joint -->
+            <joint name="left_inner_knuckle_joint">
+                <state_interface name="position">
+                    <param name="initial_value">${initial_positions['finger_joint']}</param>
+                </state_interface>
+                <state_interface name="velocity"/>
+                <state_interface name="effort">
+                    <param name="effort_limit">100.0</param>
+                </state_interface>
+            </joint>
+            <!-- right_inner_finger_joint -->
+            <joint name="right_inner_finger_joint">
+                <state_interface name="position">
+                    <param name="initial_value">${initial_positions['finger_joint']}</param>
+                </state_interface>
+                <state_interface name="velocity"/>
+                <state_interface name="effort">
+                    <param name="effort_limit">100.0</param>
+                </state_interface>
+            </joint>
+            <!-- left_inner_finger_joint -->
+            <joint name="left_inner_finger_joint">
+                <state_interface name="position">
+                    <param name="initial_value">${initial_positions['finger_joint']}</param>
+                </state_interface>
+                <state_interface name="velocity"/>
+                <state_interface name="effort">
+                    <param name="effort_limit">100.0</param>
+                </state_interface>
+            </joint>
         </ros2_control>
     </xacro:macro>
